File: PCB/NorthPoleCircuit_PCB.kicad_sch (KiCad schematic)
At the start: 56 parts, among them J1 USB_C_Receptacle_USB2.0_16P, J2 PROG, J3 PROG, U1 DRV8833PWP, U2 DRV8833PWP, U3 CH32V003FxUx, U4 CH32V003FxUx

Commit message: Add BLE audio card hardware revision
Parts:
- removed BZ1: FUET-1325H, cust_fp:FUET-1325, symbol Device:Buzzer
- removed C10: 10nF, Capacitor_SMD:C_0402_1005Metric, symbol Device:C_Small
- removed D1, D2, D3, D4: LED, LED_SMD:LED_0805_2012Metric, symbol Device:LED
- removed F1: 500mA, Fuse:Fuse_0805_2012Metric, symbol Device:Polyfuse_Small
- removed J2, J3: PROG, Connector:Tag-Connect_TC2030-IDC-NL_2x03_P1.27mm_Vertical, symbol Connector:Conn_ARM_SWD_TagConnect_TC2030-NL
- removed R3, R4: 180R, Resistor_SMD:R_0805_2012Metric, symbol Device:R_Small
- removed U1, U2: DRV8833PWP, cust_fp:HTSSOP-16-1EP_4.4x5mm_P0.65mm_EP3.4x5mm_Mask2.46x2.31mm_ThermalVias_Larger, symbol Driver_Motor:DRV8833PWP
- removed U3, U4: CH32V003FxUx, Package_DFN_QFN:QFN-20-1EP_3x3mm_P0.4mm_EP1.65x1.65mm, symbol MCU_WCH_CH32V0:CH32V003FxUx
- added AE1: Bluetooth Antenna, cust_fp:WCH_ANT_F_1_2_4G_1p0mmFR4_12p3x5p6, symbol Device:Antenna_Shield
- added BAT_PAD1: BAT_PAD, cust_fp:Battery_LiPo_500mAh_30x35x4mm_WirePads, symbol Device:R_Small
- added BT1: LiPo_1S_500mAh, cust_fp:Battery_LiPo_500mAh_30x35x4mm_Body, symbol Device:Battery_Cell
- added C11, C14, C17, C18, C20, C21, C31, C9: 10uF, Capacitor_SMD:C_1206_3216Metric, symbol Device:C_Small
- added C12, C8: 100nF, Capacitor_SMD:C_0402_1005Metric, symbol Device:C_Small
- added C16, C19, C28: 2.2uF, Capacitor_SMD:C_1206_3216Metric, symbol Device:C_Small
- added C22, C23: 22uF, Capacitor_SMD:C_1206_3216Metric, symbol Device:C_Small
- added C24, C25: 1uF, Capacitor_SMD:C_1206_3216Metric, symbol Device:C_Small
- added C4: 470nF, Capacitor_SMD:C_1206_3216Metric, symbol Device:C_Small
- added D1, D2: LESD5D5.0CT1G, Diode_SMD:D_SOD-523, symbol Device:D_TVS_Small
- added D3, D4, D5, D6, D7, D8: TZ-H1010-RGB/A-BU08UF-TA1305NA/W109, cust_fp:ws2812b_1010, symbol cust_sym:XL-1010RGBC-WS2812B
- added DM1, DM2, DP1, DP2, GND1, GND2: TestPoint_Small, TestPoint:TestPoint_Pad_D1.0mm, symbol Connector:TestPoint_Small
- added L1: ZENR3015T100M-10uH, Inductor_SMD:L_Taiyo-Yuden_NR-30xx, symbol Device:L_Small
- added L2: 1uH, Inductor_SMD:L_Wuerth_HCI-7030, symbol Device:L_Small
- added LS1: GSPK3020035PN-8R0.8W, symbol Device:Speaker
- added R11: 100kΩ, Resistor_SMD:R_0402_1005Metric, symbol Device:R_Small
- added R12, R13: 2.7kΩ, Resistor_SMD:R_0402_1005Metric, symbol Device:R_Small
- added SP_PAD1: SPK_PAD, cust_fp:Speaker_GSPK3020035PN_WirePads, symbol Device:R_Small
- added SW1, SW2: TS-1088-AR02016, Button_Switch_SMD:SW_Push_SPST_NO_Alps_SKRK, symbol Switch:SW_Push
- added SW3: TS-1187A-C-E-B, Button_Switch_SMD:SW_SPST_SKQG_WithStem, symbol Switch:SW_Push
- added U1, U3: DRV5032FADMRR, Package_SON:Texas_X2SON-4-1EP_1.1x1.4mm_P0.5mm_EP0.8x0.6mm, symbol cust_sym:DRV5032FADMRR
- added U10, U11, U9: DRV8837, Package_SON:WSON-8-1EP_2x2mm_P0.5mm_EP0.9x1.6mm, symbol Driver_Motor:DRV8837
- added U2: CH592X, Package_DFN_QFN:QFN-32-1EP_4x4mm_P0.4mm_EP2.65x2.65mm, symbol cust_sym:CH592X
- added U5: PY25Q64HA-SUH-IR, Package_SO:SOIC-8_5.3x5.3mm_P1.27mm, symbol Memory_Flash:W25X40CLSV
- added U6: WT2003H4-24SS, Package_SO:SSOP-24_3.9x8.7mm_P0.635mm, symbol cust_sym:WT2003H4-24SS
- added U7: IP5209T, Package_DFN_QFN:QFN-24-1EP_4x4mm_P0.5mm_EP2.5x2.5mm, symbol cust_sym:IP5209
- added U8: ME6211C33M5, Package_TO_SOT_SMD:SOT-23-5, symbol Regulator_Linear:ME6211C33M5
- added Y1: 32MHz, Crystal:Crystal_SMD_3225-4Pin_3.2x2.5mm, symbol Device:Crystal_GND24
- C1: value 10uF -> 4.7uF; JLCPCB (none) -> C1872; JLCPCB PN (none) -> C1872; LCSC Part (none) -> C1872; MPN C13585 -> CL31B475KAHNNNE
- C10: renamed from C16; value 100n -> 10uF; footprint Capacitor_SMD:C_0402_1005Metric -> Capacitor_SMD:C_1206_3216Metric; JLCPCB (none) -> C13585; JLCPCB PN (none) -> C13585; LCSC Part (none) -> C13585; MPN C1525 -> CL31A106KBHNNNE
- C13, C15: value 100n -> 100nF; JLCPCB (none) -> C1525; JLCPCB PN (none) -> C1525; LCSC Part (none) -> C1525; MPN C1525 -> CL05B104KO5NNNC
- C2, C3: value 10uF -> 100nF; footprint Capacitor_SMD:C_1206_3216Metric -> Capacitor_SMD:C_0402_1005Metric; JLCPCB (none) -> C1525; JLCPCB PN (none) -> C1525; LCSC Part (none) -> C1525; MPN C13585 -> CL05B104KO5NNNC
- C26: renamed from C5; JLCPCB (none) -> C50254; JLCPCB PN (none) -> C50254; LCSC Part (none) -> C50254; MPN C50254 -> CL31B225KBHNNNE
- C27: renamed from C9; JLCPCB (none) -> C50254; JLCPCB PN (none) -> C50254; LCSC Part (none) -> C50254; MPN C50254 -> CL31B225KBHNNNE
- C29: renamed from C4; JLCPCB (none) -> C13585; JLCPCB PN (none) -> C13585; LCSC Part (none) -> C13585; MPN C13585 -> CL31A106KBHNNNE
- C30: renamed from C8; JLCPCB (none) -> C13585; JLCPCB PN (none) -> C13585; LCSC Part (none) -> C13585; MPN C13585 -> CL31A106KBHNNNE
- C32: renamed from C7; JLCPCB (none) -> C13585; JLCPCB PN (none) -> C13585; LCSC Part (none) -> C13585; MPN C13585 -> CL31A106KBHNNNE
- C33: renamed from C11; JLCPCB (none) -> C13585; JLCPCB PN (none) -> C13585; LCSC Part (none) -> C13585; MPN C13585 -> CL31A106KBHNNNE
- C34: renamed from C12; JLCPCB (none) -> C13585; JLCPCB PN (none) -> C13585; LCSC Part (none) -> C13585; MPN C13585 -> CL31A106KBHNNNE
- C5: renamed from C14; value 100n -> 2.2uF; footprint Capacitor_SMD:C_0402_1005Metric -> Capacitor_SMD:C_1206_3216Metric; JLCPCB (none) -> C50254; JLCPCB PN (none) -> C50254; LCSC Part (none) -> C50254; MPN C1525 -> CL31B225KBHNNNE
- C6: value 10nF -> 100nF; JLCPCB (none) -> C1525; JLCPCB PN (none) -> C1525; LCSC Part (none) -> C1525; MPN C15195 -> CL05B104KO5NNNC
- J1: FT Position Offset (none) -> 0,1.5; JLCPCB (none) -> C165948; JLCPCB PN (none) -> C165948; LCSC Part (none) -> C165948; MPN C165948 -> TYPE-C-31-M-12
- L3: renamed from L1; value SMMS0650-101M -> 100uH; JLCPCB (none) -> C2894722; JLCPCB PN (none) -> C2894722; LCSC Part (none) -> C2894722; MPN C2894722 -> SMMS0650-101M
- L4: renamed from L2; value SMMS0650-101M -> 100uH; JLCPCB (none) -> C2894722; JLCPCB PN (none) -> C2894722; LCSC Part (none) -> C2894722; MPN C2894722 -> SMMS0650-101M
- L5: renamed from L3; value SMMS0650-101M -> 100uH; JLCPCB (none) -> C2894722; JLCPCB PN (none) -> C2894722; LCSC Part (none) -> C2894722; MPN C2894722 -> SMMS0650-101M
- R1, R2: value 5k1 -> 5.1kΩ; footprint Resistor_SMD:R_0603_1608Metric -> Resistor_SMD:R_0402_1005Metric; JLCPCB (none) -> C25905; JLCPCB PN (none) -> C25905; LCSC Part (none) -> C25905; MPN C23186 -> 0402WGF5101TCE
- R10: value 510k -> 2Ω; footprint Resistor_SMD:R_0603_1608Metric -> Resistor_SMD:R_0402_1005Metric; JLCPCB (none) -> C25157; JLCPCB PN (none) -> C25157; LCSC Part (none) -> C25157; MPN C23192 -> 0402WGJ020JTCE
- R3: renamed from R11; value 3.3k -> 3.3kΩ; JLCPCB (none) -> C25890; JLCPCB PN (none) -> C25890; LCSC Part (none) -> C25890; MPN C25890 -> 0402WGF3301TCE
- R4: renamed from R12; value 3.3k -> 3.3kΩ; JLCPCB (none) -> C25890; JLCPCB PN (none) -> C25890; LCSC Part (none) -> C25890; MPN C25890 -> 0402WGF3301TCE
- R5, R6: value 180R -> 27Ω; footprint Resistor_SMD:R_0805_2012Metric -> Resistor_SMD:R_0402_1005Metric; JLCPCB (none) -> C25100; JLCPCB PN (none) -> C25100; LCSC Part (none) -> C25100; MPN C25270 -> 0402WGF270JTCE
- R7: value 510k -> 2MΩ; footprint Resistor_SMD:R_0603_1608Metric -> Resistor_SMD:R_0805_2012Metric; JLCPCB (none) -> C40088; JLCPCB PN (none) -> C40088; LCSC Part (none) -> C40088; MPN C23192 -> 0805W8J0205T5E
- R8: value 510k -> 1MΩ; footprint Resistor_SMD:R_0603_1608Metric -> Resistor_SMD:R_0402_1005Metric; JLCPCB (none) -> C26083; JLCPCB PN (none) -> C26083; LCSC Part (none) -> C26083; MPN C23192 -> 0402WGF1004TCE
- R9: value 510k -> 10mΩ; footprint Resistor_SMD:R_0603_1608Metric -> Resistor_SMD:R_1206_3216Metric; JLCPCB (none) -> C7467248; JLCPCB PN (none) -> C7467248; LCSC Part (none) -> C7467248; MPN C23192 -> FRM121WFR010TM
- renumbered H5 to H1, H6 to H2, H9 to H5, H8 to H6, TP3 to TP1, TP4 to TP2, TP5 to TP3, TP6 to TP4
Connections:
- net +5V: now also C16.2, C20.1, C21.1, C22.1, C23.1, C24.1, C31.1, U10.1 (VM), U11.1 (VM), U6.16 (VCC), U7.16 (VOUT), U7.17 (VOUT), U8.1 (V_{IN}), U8.3 (CE), U9.1 (VM); no longer C13.1, C15.1, C3.1, C5.1, C6.1, R10.1, R3.1, R4.1, R7.1, R8.1, R9.1
- net A1_OUT: now also U10.2 (OUT1)
- net B1_OUT: now also U11.2 (OUT1)
- net G1_OUT: now also U9.2 (OUT1)
- net GND: now also C6.2, J1.SH (SHIELD), R8.2, AE1.2 (Shield), BAT_PAD1.2, BT1.2 (-), C11.2, C12.2, C14.2, C17.2, C18.2, C19.2, C20.2, C21.2, C22.2, C23.2, C24.2, C25.2, C28.1, C31.2, C4.2, C8.2, C9.2, D1.1 (A1), D2.1 (A1), D3.3 (GND), D4.3 (GND), D5.3 (GND), D6.3 (GND), D7.3 (GND), D8.3 (GND), GND1.1, GND2.1, R11.1, SW1.2, SW2.2, SW3.1, U1.3 (GND), U1.5 (GND), U10.4 (GND), U10.9 (GND), U11.4 (GND), U11.9 (GND), U2.33 (GND), U3.3 (GND), U3.5 (GND), U5.4 (GND), U6.13 (AGND), U6.17 (GND), U7.12 (PGND), U7.22 (LIGHT), U7.25 (GND), U7.7 (AGND), U8.2 (V_{SS}), U9.4 (GND), U9.9 (GND), Y1.2 (G), Y1.4 (G); no longer J1.S1 (SHIELD)
- net MUSIC: now also U2.27 (PA5); no longer R10.2
- net PWM_A1: now also U10.6 (IN1), U2.32 (PA11)
- net PWM_A2: now also U10.5 (IN2), U2.1 (PA10)
- net PWM_B1: now also U11.6 (IN1), U2.17 (PB7)
- net PWM_B2: now also U11.5 (IN2), U2.18 (PB4)
- net PWM_G1: now also U2.30 (PA13), U9.6 (IN1)
- net PWM_G2: now also U2.31 (PA12), U9.5 (IN2)
- net RUN: now also U2.8 (PA7); no longer R8.2
- net RX1: now also R12.1, U6.11 (RXD)
- net SCL: now also U2.11 (PB15), U7.24 (L1)
- net SDA: now also U2.12 (PB14), U7.1 (L2)
- net SPD++: now also U2.9 (PA8); no longer R9.2
- net SPD--: now also U2.7 (PA6); no longer R7.2
- net TX1: now also R13.1, U6.23 (TXD)
- net at L3.1: now also U9.3 (OUT2)
- net at L5.1: now also U11.3 (OUT2)
- net at J1.A6 (D+): now also J1.B6 (D+), R6.2, D1.2 (A2)
- net at J1.A7 (D-): now also J1.B7 (D-), R5.2, D2.2 (A2)
- net at L4.1: now also U10.3 (OUT2)
- net +3.3V: now reaches C26.2
- net +3.3V: now also C27.2, C3.1, C5.1, C6.1, C25.1, C28.2, D3.2 (VCC), D4.2 (VCC), D5.2 (VCC), D6.2 (VCC), D7.2 (VCC), D8.2 (VCC), U1.1 (VCC), U10.7 (~{SLEEP}), U10.8 (VCC), U11.7 (~{SLEEP}), U11.8 (VCC), U2.6 (VDD33/VIO33), U3.1 (VCC), U8.5 (V_{OUT}), U9.7 (~{SLEEP}), U9.8 (VCC)
- net LED1 renamed DN
- net DN: now also U2.16 (PB10)
- net LED4 renamed DP
- net DP: now also U2.15 (PB11)
- net VDD: no longer names the net of J1.A4 (VBUS), J1.A9 (VBUS), J1.B4 (VBUS), J1.B9 (VBUS)
- net VDD: now also R10.1, C14.1, U7.20 (VIN), U7.21 (VIN); no longer C1.1, C2.1
- new net: C1.1, C2.1, L1.1, U2.25 (VDCIA), U2.4 (VDCID)
- new net: C11.1, C13.1, C15.1, L2.1, R9.1, U7.10 (CSIN), U7.11 (CSIN_S)
- new net: BAT_PAD1.1, BT1.1 (+), C12.1, C9.1, R9.2, U7.9 (VBAT)
- new net: R12.2, U2.13 (PB13)
- new net: D6.1 (DO), D8.4 (DI)
- new net: D4.1 (DO), D6.4 (DI)
- new net: C16.1, L2.2, U7.13 (LX), U7.14 (LX), U7.15 (LX)
- new net: DM2.1, U7.18 (DM)
- new net: DP2.1, U7.19 (DP)
- new net: R11.2, U7.5 (RSET)
- new net: R7.2, R8.1, U7.6 (NTC)
- new net: SW3.2, U7.8 (KEY)
- new net: C18.1, R10.2
- new net: AE1.1 (A), U2.24 (ANT)
- new net: U5.1 (~{CS}), U6.1 (COM0)
- new net: U5.6 (CLK), U6.3 (COM2)
- new net: L1.2, U2.5 (VSW)
- new net: LS1.2, SP_PAD1.1, U6.18 (PWM+)
- new net: LS1.1, SP_PAD1.2, U6.19 (PWM-)
- new net: D4.4 (DI), D7.1 (DO)
- new net: D5.1 (DO), D7.4 (DI)
- new net: R13.2, U2.14 (PB12)
- new net: SW2.1, U2.19 (PB23)
- new net: SW1.1, U2.20 (PB22)
- new net: U2.21 (~{X32MO}), Y1.3
- new net: U2.22 (X32MI), Y1.1
- new net: C4.1, U2.23 (VINTA)
- new net: D3.1 (DO), D5.4 (DI)
- new net BUSY: U2.29 (PA14), U6.20 (LED5)
- new net DM2: DM1.1, U6.4 (ICEDAT)
- new net DO: U5.2 (DO/IO_{1}), U5.5 (DI/IO_{0}), U6.2 (COM1)
- new net DP2: DP1.1, U6.5 (ICECLK)
- new net HALL1: U1.2 (OUT), U2.2 (PB6)
- new net HALL2: U2.26 (PA4), U3.2 (OUT)
- new net INT: U2.10 (PA9), U7.2 (L3)
- new net LED: D3.4 (DI), U2.28 (PA15)
- new net VOUT: C17.1, C8.1, U5.3 (~{WP}), U5.7 (~{HOLD}), U5.8 (VCC), U6.15 (VOUT)
- new net VREG: C19.1, R3.1, R4.1, R7.1, U7.3 (VREG), U7.4 (L4)
- no-connect marks 20 -> 19
Other:
- note added: "BOOT"
- note added: "MCU"
- note added: "MP3 Audio"
- note added: "Make sure R4 & R5 are placed close to MCU"
- note added: "ON/OFF"
- note added: "POSITION REGISTRATION"
- note added: "POWER"
- note added: "RESET"
- note added: "USB"
- note added: "VSET is floating, 4.2V battery is set"
- note removed: "MCU0"
- note removed: "MCU0 GUARD TIM1_RM=00 G1 PD3 - T2CH2 G2 PC0 - T2CH3"
- note removed: "MCU0 Phases TIM1_RM=11 A1 PC4 - T1CH1 B2 PC7 - T1CH2 A2 PC5 - T1CH3 B1 PD4 - T1CH4"
- note removed: "MCU1"
- note removed: "MCU1 BUZZER TIM1_RM=01 BUZZ PD2 - T2CH3"
- note removed: "MCU1 LEDS TIM1_RM=11 LED1 PC4 - T1CH1 LED3 PC7 - T1CH2 LED2 PC5 - T1CH3 LED4 PD4 - T1CH4"
- note removed: "SMD0805B050TF - 500mA hold, 1A trip - C269104 SMD0805B075TF - 750mA hold, 1.5A trip - C269105"
- note removed: "USB POWER"
- moved on the sheet: C10, C26, C27, C29, C30, C32, C33, C34, C5, H1, H2, H5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

Commit message: Schematics and PCB update. Fiirmware v0.1
Parts:
- removed DM1, DP1, GND1: TestPoint_Small, TestPoint:TestPoint_Pad_D1.0mm, symbol Connector:TestPoint_Small
- added J3, J4: PROG, Connector:Tag-Connect_TC2030-IDC-NL_2x03_P1.27mm_Vertical, symbol Connector:Conn_ARM_SWD_TagConnect_TC2030-NL
- added R14, R15: 0Ω, Resistor_SMD:R_0402_1005Metric, symbol Device:R_Small
- added R16: 100kΩ, Resistor_SMD:R_0402_1005Metric, symbol Device:R_Small
Connections:
- net +3.3V: now also J3.1 (VCC); no longer U10.7 (~{SLEEP}), U11.7 (~{SLEEP}), U9.7 (~{SLEEP})
- net +5V: now also J4.1 (VCC)
- net DM2: now also J4.4 (SWCLK)
- net DP2: now also J4.2 (SWDIO)
- net GND: now also J3.5 (GND), J4.5 (GND), R16.2
- net SCL: now also R14.1; no longer U2.11 (PB15)
- net SDA: now also R15.1; no longer U2.12 (PB14)
- net SLEEP: now reaches U2.3 (PB0)
- net SLEEP: now also U10.7 (~{SLEEP}), U11.7 (~{SLEEP}), U9.7 (~{SLEEP}), R16.1
- new net SWDCK: J3.4 (SWCLK), R14.2, U2.11 (PB15)
- new net SWDIO: J3.2 (SWDIO), R15.2, U2.12 (PB14)
- no-connect marks 19 -> 22
Other:
- note added: "USB connector to upload MP3 files"
- moved on the sheet: C3, C6, R3, R4, U1, U3

Commit message: Final PCB update before ordering. Firmware update based on the CH592 Dev Board.
Parts:
- added +3.3V1: +3.3V, TestPoint:TestPoint_Pad_D1.5mm, symbol Connector:TestPoint
- added +5V1: +5V, TestPoint:TestPoint_Pad_D1.5mm, symbol Connector:TestPoint
- added A1: A1, TestPoint:TestPoint_Pad_D1.5mm, symbol Connector:TestPoint
- added A2: A2, TestPoint:TestPoint_Pad_D1.5mm, symbol Connector:TestPoint
- added B1: B1, TestPoint:TestPoint_Pad_D1.5mm, symbol Connector:TestPoint
- added B2: B2, TestPoint:TestPoint_Pad_D1.5mm, symbol Connector:TestPoint
- added FID1, FID2, FID3: Fiducial, Fiducial:Fiducial_0.75mm_Mask1.5mm, symbol Mechanical:Fiducial
- added G1: G1, TestPoint:TestPoint_Pad_D1.5mm, symbol Connector:TestPoint
- added G2: G2, TestPoint:TestPoint_Pad_D1.5mm, symbol Connector:TestPoint
- added GND3, HALL2: HALL2, TestPoint:TestPoint_Pad_D1.5mm, symbol Connector:TestPoint
- added HALL1: HALL1, TestPoint:TestPoint_Pad_D1.5mm, symbol Connector:TestPoint
- added LED1: LED, TestPoint:TestPoint_Pad_D1.5mm, symbol Connector:TestPoint
- added SCL1: SCL, TestPoint:TestPoint_Pad_D1.5mm, symbol Connector:TestPoint
- added SDA1: SDA, TestPoint:TestPoint_Pad_D1.5mm, symbol Connector:TestPoint
- added SLEEP1: SLEEP, TestPoint:TestPoint_Pad_D1.5mm, symbol Connector:TestPoint
Connections:
- net +3.3V: now also +3.3V1.1
- net +5V: now also +5V1.1; no longer J4.1 (VCC)
- net GND: now also GND3.1
- net HALL1: now also HALL1.1
- net HALL2: now also HALL2.1
- net LED: now also LED1.1
- net PWM_A1: now also A1.1
- net PWM_A2: now also A2.1
- net PWM_B1: now also B1.1
- net PWM_B2: now also B2.1
- net PWM_G1: now also G1.1
- net PWM_G2: now also G2.1
- net SCL: now also SCL1.1
- net SDA: now also SDA1.1
- net SLEEP: now also SLEEP1.1
- no-connect marks 22 -> 23
Other:
- note added: "FIDUCIAL"

Commit message: First tests on real PCB. PCB is alive. FW comfirms most of the functionality including BLE. Hall sensor has footprint bug. IP5209 chip still not charging the battery. LED is producing only WHITE.
Connections:
- net GND: now also U1.2 (GND), U3.2 (GND); no longer U1.3 (GND), U3.3 (GND)
- net HALL1: now also U1.4 (OUT); no longer U1.2 (OUT)
- net HALL2: now also U3.4 (OUT); no longer U3.2 (OUT)
